File: pcb/KimCard-r5.brd (EAGLE design)
At the start: 54 x 85.5 mm, 65 parts, among them U1 XMEGA16A4A, U2 MCP2221-I/SL, U4 24AA128SM

Commit message: Rev 5 almost finalized. Needs silk tuneups
Routing:
- net VCC: track 182.3 -> 189.0 mm
- net PDI_CLOCK: track 50.0 -> 48.8 mm
- net SDA: track 49.0 -> 48.1 mm
- net GND: vias 14 -> 16
- removed copper zone on layer 1, net VCC
Other:
- outline, holes or cut-outs redrawn
- board text added: "(Ind),Y"
- board text added: "(Ind,X)"
- board text added: "30mil/10%"
- board text added: "30mil/12%"
- board text added: "30mil/14%"
- board text added: "30mil/8%"
- board text added: "35mil/10%"
- board text added: "35mil/12%"
- board text added: "35mil/14%"
- board text added: "35mil/8%"
- board text added: "40mil/10%"
- board text added: "40mil/12%"
- board text added: "40mil/14%"
- board text added: "40mil/8%"
- board text added: "45mil/10%"
- board text added: "45mil/12%"
- board text added: "45mil/14%"
- board text added: "45mil/8%"
- board text added: "Abs"
- board text added: "Abs,X"
- board text added: "Abs,Y"
- board text added: "Acc"
- board text added: "BRK:00 NOP:EA CLC:18 SEC:38 CLD:D8 SED:F8 CLI:58 SEI:78 DEY:88 DEX:CA INY:C8 INX:E8 TXA:8A TYA:98 TAX:AA TAY:A8 TXS:9A TSX:BA PHP:08 PLP:28 PHA:48 PLA:68 BPL:10 BMI:30 BVS:70 BVC:50 BCS:B0 BCC:90 BEQ:F0 BNE:D0 JSR:20 RTS:60 JMP:4C JMPi:6C RTI:40 CLV:B8"
- board text added: "CLK"
- board text added: "DAT"
- board text added: "GND"
- board text added: "Imm"
- board text added: "KimCard - r5 - SmallRoomLabs.com"
- board text added: "N-Z- LDA -- A9 A5 B5 -- AD BD B9 A1 B1 N-Z- LDX -- A2 A6 -- B6 AE -- BE -- -- N-Z- LDY -- A0 A4 B4 -- AC BC -- -- -- ---- STA -- -- 85 95 -- 8D 9D 99 81 91 ---- STX -- -- 86 -- 96 8E -- -- -- -- ---- STY -- -- 84 94 -- 8C -- -- -- -- N-ZC AND -- 29 25 35 -- 2D 3D 39 21 31 N-Z- ORA -- 09 05 15 -- 0D 1D 19 01 11 N-Z- EOR -- 49 45 55 -- 4D 5D 59 41 51 NVZC ADC -- 69 65 75 -- 6D 7D 79 61 71 NVZC SBC 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"
- board text added: "PDI"
- board text added: "VCC"
- board text added: "Zp"
- board text added: "Zp,X"
- board text added: "Zp,Y"
